File: Hardware/prog-adapter/project/adapter.sch (EAGLE design)
At the start: 3 parts, among them J1 SFH11-PBPC-D10-ST-BK

Commit message: update
Other:
- note added: "MJM"
Changed lines of the file:
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@@
 <sheet>
 <plain>
+<text x="218.44" y="20.32" size="2.1844" layer="94">MJM</text>
 </plain>
 <instances>
