File: Hardware/prog-adapter/project/adapter.brd (EAGLE design)
At the start: 21 x 33 mm, 3 parts, among them J1 SFH11-PBPC-D10-ST-BK

Commit message: Update adapter.brd
Routing:
- net GND: track 10.7 -> 0.00 mm
Changed lines of the file:
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@@
 <drawing>
 <settings>
-<setting alwaysvectorfont="yes"/>
+<setting alwaysvectorfont="no"/>
 <setting verticaltext="up"/>
 </settings>
@@
 <contactref element="J1" pad="3"/>
 <contactref element="J1" pad="1"/>
-<wire x1="5.9" y1="20.32" x2="5.78" y2="20.32" width="0.1524" layer="1"/>
-<wire x1="5.78" y1="20.44" x2="5.9" y2="20.32" width="0.3048" layer="1"/>
 <polygon width="0.254" layer="1">
 <vertex x="-0.254" y="33.274"/>
@@
 </polygon>
 <contactref element="PROG1" pad="4"/>
-<wire x1="15.6338" y1="18.7098" x2="12.2528" y2="18.7098" width="0.3048" layer="1"/>
-<wire x1="12.2528" y1="18.7098" x2="10.6426" y2="20.32" width="0.3048" layer="1"/>
-<wire x1="10.6426" y1="20.32" x2="5.9" y2="20.32" width="0.3048" layer="1"/>
 </signal>
 <signal name="SWDIO">
